Commit message: edit odometry node

File: ros2_ws/src/robot_description/urdf/robot.urdf.xacro (robot description, xacro)
@@ -5,11 +5,14 @@
        Parameter
   ========================== -->
+  <xacro:arg name="wheel_radius" default="0.0745"/>
+  <xacro:arg name="wheel_width" default="0.02"/>
+  <xacro:arg name="wheel_y" default="0.11"/>
   <xacro:property name="base_length" value="0.30"/>
   <xacro:property name="base_width"  value="0.20"/>
   <xacro:property name="base_height" value="0.08"/>
-  <xacro:property name="wheel_radius" value="0.05"/>
-  <xacro:property name="wheel_width"  value="0.02"/>
+  <xacro:property name="wheel_radius" value="$(arg wheel_radius)"/>
+  <xacro:property name="wheel_width"  value="$(arg wheel_width)"/>
   <xacro:property name="wheel_x"      value="0.0"/>
-  <xacro:property name="wheel_y"      value="0.11"/>
+  <xacro:property name="wheel_y"      value="$(arg wheel_y)"/>
   <xacro:property name="wheel_z"      value="-0.05"/>
   <!-- Sensorpositionen -->

Commit message: edit positions

File: ros2_ws/src/robot_description/urdf/robot.urdf.xacro (robot description, xacro)
@@ -5,19 +5,19 @@
        Parameter
   ========================== -->
-  <xacro:arg name="wheel_radius" default="0.0745"/>
-  <xacro:arg name="wheel_width" default="0.02"/>
-  <xacro:arg name="wheel_y" default="0.11"/>
-  <xacro:property name="base_length" value="0.30"/>
-  <xacro:property name="base_width"  value="0.20"/>
-  <xacro:property name="base_height" value="0.08"/>
+  <xacro:arg name="wheel_radius" default="0.03656"/> <!-- passt -->
+  <xacro:arg name="wheel_width" default="0.0171"/> <!-- passt -->
+  <xacro:arg name="wheel_y" default="0.1606"/> <!-- passt -->
+  <xacro:property name="base_length" value="0.425"/> <!-- passt -->
+  <xacro:property name="base_width"  value="0.389"/> <!-- passt -->
+  <xacro:property name="base_height" value="0.004"/> <!-- passt -->
   <xacro:property name="wheel_radius" value="$(arg wheel_radius)"/>
   <xacro:property name="wheel_width"  value="$(arg wheel_width)"/>
-  <xacro:property name="wheel_x"      value="0.0"/>
+  <xacro:property name="wheel_x"      value="0.0"/>    <!-- passt -->
   <xacro:property name="wheel_y"      value="$(arg wheel_y)"/>
-  <xacro:property name="wheel_z"      value="-0.05"/>
+  <xacro:property name="wheel_z"      value="0.0252"/> <!-- passt -->
   <!-- Sensorpositionen -->
-  <xacro:property name="laser_x" value="0.12"/>
-  <xacro:property name="laser_y" value="0.0"/>
-  <xacro:property name="laser_z" value="0.12"/>
+  <xacro:property name="laser_x" value="0.05175"/> <!-- passt -->
+  <xacro:property name="laser_y" value="0.0"/> <!-- passt -->
+  <xacro:property name="laser_z" value="0.319"/> <!-- passt -->
   <xacro:property name="imu_x" value="0.0"/>
   <xacro:property name="imu_y" value="0.0"/>
@@ -26,7 +26,8 @@
   <xacro:property name="mag_y" value="0.0"/>
   <xacro:property name="mag_z" value="0.04"/>
-  <xacro:property name="camera_x" value="0.14"/>
-  <xacro:property name="camera_y" value="0.0"/>
-  <xacro:property name="camera_z" value="0.16"/>
+  <xacro:property name="camera_x" value="-0.03172"/> <!-- passt -->
+  <xacro:property name="camera_y" value="0.0"/> <!-- passt -->
+  <xacro:property name="camera_z" value="0.2402"/> <!-- passt -->
+  <xarco:property name="camera_p" value="0.3562"/> <!-- passt 20.41° -->
   <!-- =========================
        Farben
@@ -53,4 +54,5 @@
     <!--
     <visual>
+      <origin xyz="-0.003435 -0.000615 0" rpy="0 0 1.57079632679" /> passt
       <geometry>
         <mesh filename="package://robot_description/meshes/base.stl" scale="0.001 0.001 0.001"/>
@@ -69,5 +71,5 @@
     <origin xyz="0.10 0.12 0.05" rpy="0 0 0"/>
     <geometry>
-      <box size="0.40 0.04 0.10"/>
+      <box size="0.125 0.075 0.10"/> <!-- passt -->
     </geometry>
   </collision>
@@ -76,5 +78,5 @@
     <origin xyz="0.10 -0.12 0.05" rpy="0 0 0"/>
     <geometry>
-      <box size="0.40 0.04 0.10"/>
+      <box size="0.125 0.075 0.10"/> <!-- passt -->
     </geometry>
   </collision>
@@ -83,5 +85,5 @@
     <origin xyz="-0.10 0.0 0.05" rpy="0 0 0"/>
     <geometry>
-      <box size="0.08 0.28 0.10"/>
+      <box size="0.315 0.390 0.10"/> <!-- passt -->
     </geometry>
   </collision>
@@ -121,5 +123,5 @@
   <link name="laser_link">
     <visual>
-      <origin xyz="0 0 0" rpy="0 0 0"/>
+      <origin xyz="0 0 0.305" rpy="0 0 0"/>
       <geometry>
         <cylinder radius="0.03" length="0.04"/>
@@ -182,5 +184,5 @@
     <parent link="base_link"/>
     <child link="camera_link"/>
-    <origin xyz="${camera_x} ${camera_y} ${camera_z}" rpy="0 0 0"/>
+    <origin xyz="${camera_x} ${camera_y} ${camera_z}" rpy="0 ${camera_p} 0"/>
   </joint>
   <!-- Optischer Kamerarahmen -->

Commit message: add gripper

File: ros2_ws/src/robot_description/urdf/robot.urdf.xacro (robot description, xacro)
@@ -8,4 +8,8 @@
   <xacro:arg name="wheel_width" default="0.0171"/> <!-- passt -->
   <xacro:arg name="wheel_y" default="0.1606"/> <!-- passt -->
+  <xacro:arg name="gripper_x" default="0.3"/>
+  <xacro:arg name="gripper_y" default="0.2"/>
+  <xacro:arg name="gripper_z" default="0.1"/>
+  <xacro:arg name="gripper_yaw" default="0.0"/>
   <xacro:property name="base_length" value="0.425"/> <!-- passt -->
   <xacro:property name="base_width"  value="0.389"/> <!-- passt -->
@@ -16,4 +20,11 @@
   <xacro:property name="wheel_y"      value="$(arg wheel_y)"/>
   <xacro:property name="wheel_z"      value="0.0252"/> <!-- passt -->
+  <xacro:property name="gripper_x" value="$(arg gripper_x)"/>
+  <xacro:property name="gripper_y" value="$(arg gripper_y)"/>
+  <xacro:property name="gripper_z" value="$(arg gripper_z)"/>
+  <xacro:property name="gripper_yaw" value="$(arg gripper_yaw)"/>
+  <xacro:property name="gripper_length" value="0.1"/>
+  <xacro:property name="gripper_width" value="0.1"/>
+  <xacro:property name="gripper_height" value="0.1"/>
   <!-- Sensorpositionen -->
   <xacro:property name="laser_x" value="0.05175"/> <!-- passt -->
@@ -29,5 +40,5 @@
   <xacro:property name="camera_y" value="0.0"/> <!-- passt -->
   <xacro:property name="camera_z" value="0.2402"/> <!-- passt -->
-  <xarco:property name="camera_p" value="0.3562"/> <!-- passt 20.41° -->
+  <xacro:property name="camera_p" value="0.3562"/> <!-- passt 20.41° -->
   <!-- =========================
        Farben
@@ -118,4 +129,43 @@
   <xacro:wheel name="left_wheel_link"  x="${wheel_x}" y="${wheel_y}"  z="${wheel_z}"/>
   <xacro:wheel name="right_wheel_link" x="${wheel_x}" y="-${wheel_y}" z="${wheel_z}"/>
+<!-- =========================
+       Gripper Macro
+  ========================== -->
+  <xacro:macro name="gripper" params="name x y z yaw">
+    <link name="${name}">
+      <visual>
+        <origin xyz="${gripper_length/2.0} 0 0" rpy="0 0 0"/>
+        <geometry>
+          <box size="${gripper_length} ${gripper_width} ${gripper_height}"/>
+        </geometry>
+        <material name="black"/>
+      </visual>
+      <!--
+      <visual>
+        <origin xyz="0 0 0" rpy="0 0 0" />
+        <geometry>
+          <mesh filename="package://robot_description/meshes/base.stl" scale="0.001 0.001 0.001"/>
+        </geometry>
+        <material name="black"/>
+      </visual>
+    -->
+      <collision>
+        <origin xyz="${gripper_length/2.0} 0 0" rpy="0 0 0"/>
+        <geometry>
+          <box size="${gripper_length} ${gripper_width} ${gripper_height}"/>
+        </geometry>
+      </collision>
+    </link>
+    <joint name="${name}_joint" type="revolute">
+      <parent link="base_link"/>
+      <child link="${name}"/>
+      <origin xyz="${x} ${y} ${z}" rpy="0 0 ${yaw}"/>
+      <axis xyz="0 0 1"/>
+      <limit lower="0" upper="3.145" effort="1.0" velocity="1.0"/>
+    </joint>
+  </xacro:macro>
+  <!-- Greifer -->
+  <xacro:gripper name="left_gripper_link" x="${gripper_x}" y="${gripper_y}" z="${gripper_z}" yaw="${gripper_yaw}"/>
+  <xacro:gripper name="right_gripper_link" x="${gripper_x}" y="-${gripper_y}" z="${gripper_z}" yaw="-${gripper_yaw}"/>
   <!-- =========================
        LiDAR
@@ -123,5 +173,5 @@
   <link name="laser_link">
     <visual>
-      <origin xyz="0 0 0.305" rpy="0 0 0"/>
+      <origin xyz="0 0 0" rpy="0 0 0"/>
       <geometry>
         <cylinder radius="0.03" length="0.04"/>

Commit message: add meshes and edit urdf for meshes

File: ros2_ws/src/robot_description/urdf/robot.urdf.xacro (robot description, xacro)
@@ -63,13 +63,12 @@
   ========================== -->
   <link name="base_link">
+    <visual>
+      <origin xyz="-0.003435 -0.000615 0" rpy="0 0 1.57079632679" /> passt
+      <geometry>
+        <mesh filename="package://robot_description/meshes/BRT7K.stl" scale="0.001 0.001 0.001"/>
+      </geometry>
+    </visual>
     <!--
     <visual>
-      <origin xyz="-0.003435 -0.000615 0" rpy="0 0 1.57079632679" /> passt
-      <geometry>
-        <mesh filename="package://robot_description/meshes/base.stl" scale="0.001 0.001 0.001"/>
-      </geometry>
-    </visual>
-    -->
-    <visual>
       <origin xyz="0 0 ${base_height/2.0}" rpy="0 0 0"/>
       <geometry>
@@ -78,4 +77,5 @@
       <material name="blue"/>
     </visual>
+  -->
    <!-- linker U-Schenkel -->
   <collision>
@@ -132,40 +132,44 @@
        Gripper Macro
   ========================== -->
-  <xacro:macro name="gripper" params="name x y z yaw">
-    <link name="${name}">
-      <visual>
-        <origin xyz="${gripper_length/2.0} 0 0" rpy="0 0 0"/>
-        <geometry>
-          <box size="${gripper_length} ${gripper_width} ${gripper_height}"/>
-        </geometry>
-        <material name="black"/>
-      </visual>
-      <!--
-      <visual>
-        <origin xyz="0 0 0" rpy="0 0 0" />
-        <geometry>
-          <mesh filename="package://robot_description/meshes/base.stl" scale="0.001 0.001 0.001"/>
-        </geometry>
-        <material name="black"/>
-      </visual>
-    -->
-      <collision>
-        <origin xyz="${gripper_length/2.0} 0 0" rpy="0 0 0"/>
-        <geometry>
-          <box size="${gripper_length} ${gripper_width} ${gripper_height}"/>
-        </geometry>
-      </collision>
-    </link>
-    <joint name="${name}_joint" type="revolute">
-      <parent link="base_link"/>
-      <child link="${name}"/>
-      <origin xyz="${x} ${y} ${z}" rpy="0 0 ${yaw}"/>
-      <axis xyz="0 0 1"/>
-      <limit lower="0" upper="3.145" effort="1.0" velocity="1.0"/>
-    </joint>
-  </xacro:macro>
+  <xacro:macro name="gripper" params="name x y z yaw mesh_file">
+  <link name="${name}">
+    <visual>
+      <origin xyz="0 0 0" rpy="0 0 0"/>
+      <geometry>
+        <mesh filename="package://robot_description/meshes/${mesh_file}"
+              scale="0.001 0.001 0.001"/>
+      </geometry>
+      <material name="black"/>
+    </visual>
+    <collision>
+      <origin xyz="${gripper_length/2.0} 0 0" rpy="0 0 0"/>
+      <geometry>
+        <box size="${gripper_length} ${gripper_width} ${gripper_height}"/>
+      </geometry>
+    </collision>
+  </link>
+  <joint name="${name}_joint" type="revolute">
+    <parent link="base_link"/>
+    <child link="${name}"/>
+    <origin xyz="${x} ${y} ${z}" rpy="0 0 ${yaw}"/>
+    <axis xyz="0 0 1"/>
+    <limit lower="0" upper="3.145" effort="1.0" velocity="1.0"/>
+  </joint>
+</xacro:macro>
   <!-- Greifer -->
-  <xacro:gripper name="left_gripper_link" x="${gripper_x}" y="${gripper_y}" z="${gripper_z}" yaw="${gripper_yaw}"/>
-  <xacro:gripper name="right_gripper_link" x="${gripper_x}" y="-${gripper_y}" z="${gripper_z}" yaw="-${gripper_yaw}"/>
+  <xacro:gripper
+  name="left_gripper_link"
+  x="${gripper_x}"
+  y="${gripper_y}"
+  z="${gripper_z}"
+  yaw="${gripper_yaw}"
+  mesh_file="gripper_left.stl"/>
+<xacro:gripper
+  name="right_gripper_link"
+  x="${gripper_x}"
+  y="-${gripper_y}"
+  z="${gripper_z}"
+  yaw="-${gripper_yaw}"
+  mesh_file="gripper_right.stl"/>
   <!-- =========================
        LiDAR

Commit message: fix tf links

File: ros2_ws/src/robot_description/urdf/robot.urdf.xacro (robot description, xacro)
@@ -28,7 +28,7 @@
   <xacro:property name="gripper_height" value="0.1"/>
   <!-- Sensorpositionen -->
-  <xacro:property name="laser_x" value="0.05175"/> <!-- passt -->
+  <xacro:property name="laser_x" value="0.0"/> <!-- passt -->
   <xacro:property name="laser_y" value="0.0"/> <!-- passt -->
-  <xacro:property name="laser_z" value="0.319"/> <!-- passt -->
+  <xacro:property name="laser_z" value="0.29"/> <!-- passt -->
   <xacro:property name="imu_x" value="0.0"/>
   <xacro:property name="imu_y" value="0.0"/>

Commit message: add softstart for drive wheels, add percent for finish in frontierexplorer, set the whole odomtree to 5 Hz, correct typo in urdf, add single services for hardware nodes

File: ros2_ws/src/robot_description/urdf/robot.urdf.xacro (robot description, xacro)
@@ -31,4 +31,5 @@
   <xacro:property name="laser_y" value="0.0"/> <!-- passt -->
   <xacro:property name="laser_z" value="0.29"/> <!-- passt -->
+  <xacro:property name="laser_yaw" value="1.57079632679"/>
   <xacro:property name="imu_x" value="0.0"/>
   <xacro:property name="imu_y" value="0.0"/>
@@ -187,5 +188,5 @@
     <parent link="base_link"/>
     <child link="laser_link"/>
-    <origin xyz="${laser_x} ${laser_y} ${laser_z}" rpy="0 0 0"/>
+    <origin xyz="${laser_x} ${laser_y} ${laser_z}" rpy="0 0 ${laser_yaw}"/>
   </joint>
   <!-- =========================

Commit message: fix froniter explorer params

File: ros2_ws/src/robot_description/urdf/robot.urdf.xacro (robot description, xacro)
@@ -31,5 +31,5 @@
   <xacro:property name="laser_y" value="0.0"/> <!-- passt -->
   <xacro:property name="laser_z" value="0.29"/> <!-- passt -->
-  <xacro:property name="laser_yaw" value="1.57079632679"/>
+  <xacro:property name="laser_yaw" value="0"/>
   <xacro:property name="imu_x" value="0.0"/>
   <xacro:property name="imu_y" value="0.0"/>

Commit message: fix lidar yaw

File: ros2_ws/src/robot_description/urdf/robot.urdf.xacro (robot description, xacro)
@@ -31,5 +31,5 @@
   <xacro:property name="laser_y" value="0.0"/> <!-- passt -->
   <xacro:property name="laser_z" value="0.29"/> <!-- passt -->
-  <xacro:property name="laser_yaw" value="0"/>
+  <xacro:property name="laser_yaw" value="1.57079632679"/>
   <xacro:property name="imu_x" value="0.0"/>
   <xacro:property name="imu_y" value="0.0"/>

Commit message: fix robot description geometry and odometry dimensions

File: ros2_ws/src/robot_description/urdf/robot.urdf.xacro (robot description, xacro)
@@ -31,5 +31,5 @@
   <xacro:property name="laser_y" value="0.0"/> <!-- passt -->
   <xacro:property name="laser_z" value="0.29"/> <!-- passt -->
-  <xacro:property name="laser_yaw" value="1.57079632679"/>
+  <xacro:property name="laser_yaw" value="-1.57079632679"/>
   <xacro:property name="imu_x" value="0.0"/>
   <xacro:property name="imu_y" value="0.0"/>
@@ -65,5 +65,5 @@
   <link name="base_link">
     <visual>
-      <origin xyz="-0.003435 -0.000615 0" rpy="0 0 1.57079632679" /> passt
+      <origin xyz="-0.003435 -0.000615 0" rpy="0 0 1.57079632679"/>
       <geometry>
         <mesh filename="package://robot_description/meshes/BRT7K.stl" scale="0.001 0.001 0.001"/>
@@ -133,8 +133,8 @@
        Gripper Macro
   ========================== -->
-  <xacro:macro name="gripper" params="name x y z yaw mesh_file">
+  <xacro:macro name="gripper" params="name x y z yaw mesh_file visual_x visual_y visual_z">
   <link name="${name}">
     <visual>
-      <origin xyz="0 0 0" rpy="0 0 0"/>
+      <origin xyz="${visual_x} ${visual_y} ${visual_z}" rpy="0 0 0"/>
       <geometry>
         <mesh filename="package://robot_description/meshes/${mesh_file}"
@@ -165,5 +165,8 @@
   z="${gripper_z}"
   yaw="${gripper_yaw}"
-  mesh_file="gripper_left.stl"/>
+  mesh_file="gripper_left.stl"
+  visual_x="0.106920"
+  visual_y="-0.165493"
+  visual_z="-0.031400"/>
 <xacro:gripper
   name="right_gripper_link"
@@ -172,5 +175,8 @@
   z="${gripper_z}"
   yaw="-${gripper_yaw}"
-  mesh_file="gripper_right.stl"/>
+  mesh_file="gripper_right.stl"
+  visual_x="-0.106894"
+  visual_y="-0.165477"
+  visual_z="-0.019400"/>
   <!-- =========================
        LiDAR

Commit message: Rotate lidar frame 180 degrees

File: ros2_ws/src/robot_description/urdf/robot.urdf.xacro (robot description, xacro)
@@ -31,5 +31,5 @@
   <xacro:property name="laser_y" value="0.0"/> <!-- passt -->
   <xacro:property name="laser_z" value="0.29"/> <!-- passt -->
-  <xacro:property name="laser_yaw" value="-1.57079632679"/>
+  <xacro:property name="laser_yaw" value="1.57079632679"/>
   <xacro:property name="imu_x" value="0.0"/>
   <xacro:property name="imu_y" value="0.0"/>

Commit message: Invert lidar scan instead of rotating frame

File: ros2_ws/src/robot_description/urdf/robot.urdf.xacro (robot description, xacro)
@@ -31,5 +31,5 @@
   <xacro:property name="laser_y" value="0.0"/> <!-- passt -->
   <xacro:property name="laser_z" value="0.29"/> <!-- passt -->
-  <xacro:property name="laser_yaw" value="1.57079632679"/>
+  <xacro:property name="laser_yaw" value="-1.57079632679"/>
   <xacro:property name="imu_x" value="0.0"/>
   <xacro:property name="imu_y" value="0.0"/>

Commit message: Flip lidar TF roll

File: ros2_ws/src/robot_description/urdf/robot.urdf.xacro (robot description, xacro)
@@ -31,5 +31,6 @@
   <xacro:property name="laser_y" value="0.0"/> <!-- passt -->
   <xacro:property name="laser_z" value="0.29"/> <!-- passt -->
-  <xacro:property name="laser_yaw" value="-1.57079632679"/>
+  <xacro:property name="laser_roll" value="3.14159265359"/>
+  <xacro:property name="laser_yaw" value="0.0"/>
   <xacro:property name="imu_x" value="0.0"/>
   <xacro:property name="imu_y" value="0.0"/>
@@ -194,5 +195,5 @@
     <parent link="base_link"/>
     <child link="laser_link"/>
-    <origin xyz="${laser_x} ${laser_y} ${laser_z}" rpy="0 0 ${laser_yaw}"/>
+    <origin xyz="${laser_x} ${laser_y} ${laser_z}" rpy="${laser_roll} 0 ${laser_yaw}"/>
   </joint>
   <!-- =========================

Commit message: Adjust base collision geometry

File: ros2_ws/src/robot_description/urdf/robot.urdf.xacro (robot description, xacro)
@@ -5,19 +5,19 @@
        Parameter
   ========================== -->
-  <xacro:arg name="wheel_radius" default="0.03656"/> <!-- passt -->
-  <xacro:arg name="wheel_width" default="0.0171"/> <!-- passt -->
-  <xacro:arg name="wheel_y" default="0.1606"/> <!-- passt -->
+  <xacro:arg name="wheel_radius" default="0.03656"/>
+  <xacro:arg name="wheel_width" default="0.0171"/>
+  <xacro:arg name="wheel_y" default="0.1606"/>
   <xacro:arg name="gripper_x" default="0.3"/>
   <xacro:arg name="gripper_y" default="0.2"/>
   <xacro:arg name="gripper_z" default="0.1"/>
   <xacro:arg name="gripper_yaw" default="0.0"/>
-  <xacro:property name="base_length" value="0.425"/> <!-- passt -->
-  <xacro:property name="base_width"  value="0.389"/> <!-- passt -->
-  <xacro:property name="base_height" value="0.004"/> <!-- passt -->
+  <xacro:property name="base_length" value="0.425"/>
+  <xacro:property name="base_width"  value="0.389"/>
+  <xacro:property name="base_height" value="0.004"/>
   <xacro:property name="wheel_radius" value="$(arg wheel_radius)"/>
   <xacro:property name="wheel_width"  value="$(arg wheel_width)"/>
-  <xacro:property name="wheel_x"      value="0.0"/>    <!-- passt -->
+  <xacro:property name="wheel_x"      value="0.0"/>
   <xacro:property name="wheel_y"      value="$(arg wheel_y)"/>
-  <xacro:property name="wheel_z"      value="0.0252"/> <!-- passt -->
+  <xacro:property name="wheel_z"      value="0.0252"/>
   <xacro:property name="gripper_x" value="$(arg gripper_x)"/>
   <xacro:property name="gripper_y" value="$(arg gripper_y)"/>
@@ -28,7 +28,7 @@
   <xacro:property name="gripper_height" value="0.1"/>
   <!-- Sensorpositionen -->
-  <xacro:property name="laser_x" value="0.0"/> <!-- passt -->
-  <xacro:property name="laser_y" value="0.0"/> <!-- passt -->
-  <xacro:property name="laser_z" value="0.29"/> <!-- passt -->
+  <xacro:property name="laser_x" value="0.0"/>
+  <xacro:property name="laser_y" value="0.0"/>
+  <xacro:property name="laser_z" value="0.29"/>
   <xacro:property name="laser_roll" value="3.14159265359"/>
   <xacro:property name="laser_yaw" value="0.0"/>
@@ -39,8 +39,8 @@
   <xacro:property name="mag_y" value="0.0"/>
   <xacro:property name="mag_z" value="0.04"/>
-  <xacro:property name="camera_x" value="-0.03172"/> <!-- passt -->
-  <xacro:property name="camera_y" value="0.0"/> <!-- passt -->
-  <xacro:property name="camera_z" value="0.2402"/> <!-- passt -->
-  <xacro:property name="camera_p" value="0.3562"/> <!-- passt 20.41° -->
+  <xacro:property name="camera_x" value="-0.03172"/>
+  <xacro:property name="camera_y" value="0.0"/>
+  <xacro:property name="camera_z" value="0.2402"/>
+  <xacro:property name="camera_p" value="0.3562"/>
   <!-- =========================
        Farben
@@ -82,14 +82,14 @@
    <!-- linker U-Schenkel -->
   <collision>
-    <origin xyz="0.10 0.12 0.05" rpy="0 0 0"/>
+    <origin xyz="0.215 0.155 0.05" rpy="0 0 0"/>
     <geometry>
-      <box size="0.125 0.075 0.10"/> <!-- passt -->
+      <box size="0.22 0.09 0.10"/> <!-- passt -->
     </geometry>
   </collision>
   <!-- rechter U-Schenkel -->
   <collision>
-    <origin xyz="0.10 -0.12 0.05" rpy="0 0 0"/>
+    <origin xyz="0.215 -0.155 0.05" rpy="0 0 0"/>
     <geometry>
-      <box size="0.125 0.075 0.10"/> <!-- passt -->
+      <box size="0.22 0.09 0.10"/> <!-- passt -->
     </geometry>
   </collision>
@@ -98,5 +98,5 @@
     <origin xyz="-0.10 0.0 0.05" rpy="0 0 0"/>
     <geometry>
-      <box size="0.315 0.390 0.10"/> <!-- passt -->
+      <box size="0.41 0.4 0.10"/> <!-- passt -->
     </geometry>
   </collision>

Commit message: change wheel params in urdf

File: ros2_ws/src/robot_description/urdf/robot.urdf.xacro (robot description, xacro)
@@ -5,7 +5,7 @@
        Parameter
   ========================== -->
-  <xacro:arg name="wheel_radius" default="0.03656"/>
-  <xacro:arg name="wheel_width" default="0.0171"/>
-  <xacro:arg name="wheel_y" default="0.1606"/>
+  <xacro:arg name="wheel_radius" default="0.03660"/>
+  <xacro:arg name="wheel_width" default="0.0200"/>
+  <xacro:arg name="wheel_y" default="0.2110"/>
   <xacro:arg name="gripper_x" default="0.3"/>
   <xacro:arg name="gripper_y" default="0.2"/>
@@ -19,5 +19,5 @@
   <xacro:property name="wheel_x"      value="0.0"/>
   <xacro:property name="wheel_y"      value="$(arg wheel_y)"/>
-  <xacro:property name="wheel_z"      value="0.0252"/>
+  <xacro:property name="wheel_z"      value="0.0"/>
   <xacro:property name="gripper_x" value="$(arg gripper_x)"/>
   <xacro:property name="gripper_y" value="$(arg gripper_y)"/>

Commit message: add base footprint

File: ros2_ws/src/robot_description/urdf/robot.urdf.xacro (robot description, xacro)
@@ -102,4 +102,11 @@
   </collision>
 </link>
+<link name="base_footprint">
+  </link>
+  <joint name="base_footprint" type="fixed">
+    <parent link="base_link"/>
+    <child link="base_footprint"/>
+    <origin xyz="0 0 0" rpy="0 0 0"/>
+  </joint>
   <!-- =========================
        Wheel Macro
